Commit message: corrected apple.xacro

File: kuka_description/urdf/models/apple.xacro (robot description, xacro)
@@ -1,276 +1,23 @@
 <?xml version="1.0"?>
-<robot xmlns:xacro="http://www.ros.org/wiki/xacro">
-    <!-- robot as extracted via https://github.com/syuntoku14/fusion2urdf -->
-    <xacro:macro name="iiwa7"
-        params="robot_name:=^|lbr mode:=^|mock system_config_path:=^|'$(find lbr_description)/ros2_control/lbr_system_config.yaml' initial_joint_positions_path:=^|'$(find lbr_description)/ros2_control/initial_joint_positions.yaml'">
-        <!-- includes -->
-        <xacro:include filename="$(find lbr_description)/gazebo/lbr_gazebo.xacro" />
-        <xacro:include filename="$(find lbr_description)/ros2_control/lbr_system_interface.xacro" />
-        <!-- joint limits via yaml -->
-        <xacro:property name="joint_limits_path"
-            value="$(find lbr_description)/urdf/iiwa7/joint_limits.yaml" />
-        <xacro:property name="joint_limits" value="${xacro.load_yaml(joint_limits_path)}" />
-        <!-- constants -->
-        <xacro:property name="PI" value="3.1415926535897931" />
-        <xacro:property name="joint_damping" value="10.0" />
-        <xacro:property name="joint_friction" value="0.1" />
-        <!-- macros for gazebo / mock / hardware -->
-        <xacro:lbr_gazebo robot_name="${robot_name}" />
-        <xacro:lbr_system_interface
-            robot_name="${robot_name}"
-            mode="${mode}"
-            joint_limits="${joint_limits}"
-            system_config_path="${system_config_path}"
-            initial_joint_positions_path="${initial_joint_positions_path}" />
-        <link name="${robot_name}_link_0">
-            <inertial>
-                <origin rpy="0 0 0" xyz="-0.012857 0.0 0.069964" />
-                <mass value="4.855658" />
-                <inertia ixx="0.017839" ixy="0.0" ixz="0.000781" iyy="0.022294" iyz="0.0"
-                    izz="0.021334" />
-            </inertial>
-            <visual>
-                <origin rpy="0 0 0" xyz="0 0 0" />
-                <geometry>
-                    <mesh filename="package://lbr_description/meshes/iiwa7/visual/link_0.dae" />
-                </geometry>
-            </visual>
-            <collision>
-                <origin rpy="0 0 0" xyz="0 0 0" />
-                <geometry>
-                    <mesh filename="package://lbr_description/meshes/iiwa7/collision/link_0.stl" />
-                </geometry>
-            </collision>
-        </link>
-        <joint name="${robot_name}_A1" type="revolute">
-            <origin rpy="0 0 0" xyz="0.0 0.0 0.1475" />
-            <parent link="${robot_name}_link_0" />
-            <child link="${robot_name}_link_1" />
-            <axis xyz="0.0 0.0 1.0" />
-            <limit
-                effort="${joint_limits['A1']['effort']}"
-                lower="${joint_limits['A1']['lower'] * PI / 180}"
-                upper="${joint_limits['A1']['upper'] * PI / 180}"
-                velocity="${joint_limits['A1']['velocity'] * PI / 180}" />
-            <dynamics damping="${joint_damping}" friction="${joint_friction}" />
-        </joint>
-        <link name="${robot_name}_link_1">
-            <inertial>
-                <origin rpy="0 0 0" xyz="0.0 -0.034819 0.123299" />
-                <mass value="3.394011" />
-                <inertia ixx="0.021383" ixy="0.0" ixz="0.0" iyy="0.020403" iyz="0.003797"
-                    izz="0.007563" />
-            </inertial>
-            <visual>
-                <origin rpy="0 0 0" xyz="0.0 0.0 -0.1475" />
-                <geometry>
-                    <mesh filename="package://lbr_description/meshes/iiwa7/visual/link_1.dae" />
-                </geometry>
-            </visual>
-            <collision>
-                <origin rpy="0 0 0" xyz="0.0 0.0 -0.1475" />
-                <geometry>
-                    <mesh filename="package://lbr_description/meshes/iiwa7/collision/link_1.stl" />
-                </geometry>
-            </collision>
-        </link>
-        <joint name="${robot_name}_A2" type="revolute">
-            <origin rpy="0 0 0" xyz="0.0 -0.0105 0.1925" />
-            <parent link="${robot_name}_link_1" />
-            <child link="${robot_name}_link_2" />
-            <axis xyz="0.0 1.0 0.0" />
-            <limit
-                effort="${joint_limits['A2']['effort']}"
-                lower="${joint_limits['A2']['lower'] * PI / 180}"
-                upper="${joint_limits['A2']['upper'] * PI / 180}"
-                velocity="${joint_limits['A2']['velocity'] * PI / 180}" />
-            <dynamics damping="${joint_damping}" friction="${joint_friction}" />
-        </joint>
-        <link name="${robot_name}_link_2">
-            <inertial>
-                <origin rpy="0 0 0" xyz="0.0 0.039793 0.086944" />
-                <mass value="4.031991" />
-                <inertia ixx="0.031697" ixy="0.0" ixz="0.0" iyy="0.03008" iyz="0.005889"
-                    izz="0.009666" />
-            </inertial>
-            <visual>
-                <origin rpy="0 0 0" xyz="0.0 0.0105 -0.34" />
-                <geometry>
-                    <mesh filename="package://lbr_description/meshes/iiwa7/visual/link_2.dae" />
-                </geometry>
-            </visual>
-            <collision>
-                <origin rpy="0 0 0" xyz="0.0 0.0105 -0.34" />
-                <geometry>
-                    <mesh filename="package://lbr_description/meshes/iiwa7/collision/link_2.stl" />
-                </geometry>
-            </collision>
-        </link>
-        <joint name="${robot_name}_A3" type="revolute">
-            <origin rpy="0 0 0" xyz="0.0 0.0105 0.2075" />
-            <parent link="${robot_name}_link_2" />
-            <child link="${robot_name}_link_3" />
-            <axis xyz="0.0 0.0 1.0" />
-            <limit
-                effort="${joint_limits['A3']['effort']}"
-                lower="${joint_limits['A3']['lower'] * PI / 180}"
-                upper="${joint_limits['A3']['upper'] * PI / 180}"
-                velocity="${joint_limits['A3']['velocity'] * PI / 180}" />
-            <dynamics damping="${joint_damping}" friction="${joint_friction}" />
-        </joint>
-        <link name="${robot_name}_link_3">
-            <inertial>
-                <origin rpy="0 0 0" xyz="0.0 0.034819 0.123299" />
-                <mass value="3.394011" />
-                <inertia ixx="0.021383" ixy="0.0" ixz="0.0" iyy="0.020403" iyz="-0.003797"
-                    izz="0.007563" />
-            </inertial>
-            <visual>
-                <origin rpy="0 0 0" xyz="0.0 0.0 -0.5475" />
-                <geometry>
-                    <mesh filename="package://lbr_description/meshes/iiwa7/visual/link_3.dae" />
-                </geometry>
-            </visual>
-            <collision>
-                <origin rpy="0 0 0" xyz="0.0 0.0 -0.5475" />
-                <geometry>
-                    <mesh filename="package://lbr_description/meshes/iiwa7/collision/link_3.stl" />
-                </geometry>
-            </collision>
-        </link>
-        <joint name="${robot_name}_A4" type="revolute">
-            <origin rpy="0 0 0" xyz="0.0 0.0105 0.1925" />
-            <parent link="${robot_name}_link_3" />
-            <child link="${robot_name}_link_4" />
-            <axis xyz="0.0 -1.0 0.0" />
-            <limit
-                effort="${joint_limits['A4']['effort']}"
-                lower="${joint_limits['A4']['lower'] * PI / 180}"
-                upper="${joint_limits['A4']['upper'] * PI / 180}"
-                velocity="${joint_limits['A4']['velocity'] * PI / 180}" />
-            <dynamics damping="${joint_damping}" friction="${joint_friction}" />
-        </joint>
-        <link name="${robot_name}_link_4">
-            <inertial>
-                <origin rpy="0 0 0" xyz="0.0 -0.039793 0.086944" />
-                <mass value="4.031989" />
-                <inertia ixx="0.031695" ixy="0.0" ixz="0.0" iyy="0.030079" iyz="-0.005889"
-                    izz="0.009665" />
-            </inertial>
-            <visual>
-                <origin rpy="0 0 0" xyz="0.0 -0.0105 -0.74" />
-                <geometry>
-                    <mesh filename="package://lbr_description/meshes/iiwa7/visual/link_4.dae" />
-                </geometry>
-            </visual>
-            <collision>
-                <origin rpy="0 0 0" xyz="0.0 -0.0105 -0.74" />
-                <geometry>
-                    <mesh filename="package://lbr_description/meshes/iiwa7/collision/link_4.stl" />
-                </geometry>
-            </collision>
-        </link>
-        <joint name="${robot_name}_A5" type="revolute">
-            <origin rpy="0 0 0" xyz="0.0 -0.0105 0.2075" />
-            <parent link="${robot_name}_link_4" />
-            <child link="${robot_name}_link_5" />
-            <axis xyz="0.0 0.0 1.0" />
-            <limit
-                effort="${joint_limits['A5']['effort']}"
-                lower="${joint_limits['A5']['lower'] * PI / 180}"
-                upper="${joint_limits['A5']['upper'] * PI / 180}"
-                velocity="${joint_limits['A5']['velocity'] * PI / 180}" />
-            <dynamics damping="${joint_damping}" friction="${joint_friction}" />
-        </joint>
-        <link name="${robot_name}_link_5">
-            <inertial>
-                <origin rpy="0 0 0" xyz="0.0 -0.029824 0.076267" />
-                <mass value="1.529239" />
-                <inertia ixx="0.008485" ixy="0.0" ixz="0.0" iyy="0.007136" iyz="0.002806"
-                    izz="0.003848" />
-            </inertial>
-            <visual>
-                <origin rpy="0 0 0" xyz="0.0 0.0 -0.9475" />
-                <geometry>
-                    <mesh filename="package://lbr_description/meshes/iiwa7/visual/link_5.dae" />
-                </geometry>
-            </visual>
-            <collision>
-                <origin rpy="0 0 0" xyz="0.0 0.0 -0.9475" />
-                <geometry>
-                    <mesh filename="package://lbr_description/meshes/iiwa7/collision/link_5.stl" />
-                </geometry>
-            </collision>
-        </link>
-        <joint name="${robot_name}_A6" type="revolute">
-            <origin rpy="0 0 0" xyz="0.0 -0.0707 0.1925" />
-            <parent link="${robot_name}_link_5" />
-            <child link="${robot_name}_link_6" />
-            <axis xyz="0.0 1.0 0.0" />
-            <limit
-                effort="${joint_limits['A6']['effort']}"
-                lower="${joint_limits['A6']['lower'] * PI / 180}"
-                upper="${joint_limits['A6']['upper'] * PI / 180}"
-                velocity="${joint_limits['A6']['velocity'] * PI / 180}" />
-            <dynamics damping="${joint_damping}" friction="${joint_friction}" />
-        </joint>
-        <link name="${robot_name}_link_6">
-            <inertial>
-                <origin rpy="0 0 0" xyz="0.0 0.07102 0.00495" />
-                <mass value="2.403626" />
-                <inertia ixx="0.007067" ixy="0.0" ixz="0.0" iyy="0.006804" iyz="0.000311"
-                    izz="0.004629" />
-            </inertial>
-            <visual>
-                <origin rpy="0 0 0" xyz="0.0 0.0707 -1.14" />
-                <geometry>
-                    <mesh filename="package://lbr_description/meshes/iiwa7/visual/link_6.dae" />
-                </geometry>
-            </visual>
-            <collision>
-                <origin rpy="0 0 0" xyz="0.0 0.0707 -1.14" />
-                <geometry>
-                    <mesh filename="package://lbr_description/meshes/iiwa7/collision/link_6.stl" />
-                </geometry>
-            </collision>
-        </link>
-        <joint name="${robot_name}_A7" type="revolute">
-            <origin rpy="0 0 0" xyz="0.0 0.0707 0.091" />
-            <parent link="${robot_name}_link_6" />
-            <child link="${robot_name}_link_7" />
-            <axis xyz="0.0 0.0 1.0" />
-            <limit
-                effort="${joint_limits['A7']['effort']}"
-                lower="${joint_limits['A7']['lower'] * PI / 180}"
-                upper="${joint_limits['A7']['upper'] * PI / 180}"
-                velocity="${joint_limits['A7']['velocity'] * PI / 180}" />
-            <dynamics damping="${joint_damping}" friction="${joint_friction}" />
-        </joint>
-        <link name="${robot_name}_link_7">
-            <inertial>
-                <origin rpy="0 0 0" xyz="3.0000e-06 -2.0000e-06 1.3782e-02" />
-                <mass value="0.259474" />
-                <inertia ixx="0.000171" ixy="0.0" ixz="0.0" iyy="0.000171" iyz="0.0" izz="0.000299" />
-            </inertial>
-            <visual>
-                <origin rpy="0 0 0" xyz="0.0 0.0 -1.231" />
-                <geometry>
-                    <mesh filename="package://lbr_description/meshes/iiwa7/visual/link_7.dae" />
-                </geometry>
-            </visual>
-            <collision>
-                <origin rpy="0 0 0" xyz="0.0 0.0 -1.231" />
-                <geometry>
-                    <mesh filename="package://lbr_description/meshes/iiwa7/collision/link_7.stl" />
-                </geometry>
-            </collision>
-        </link>
-        <joint name="${robot_name}_joint_ee" type="fixed">
-            <parent link="${robot_name}_link_7" />
-            <child link="${robot_name}_link_ee" />
-            <origin xyz="0 0 0.035" rpy="0 0 0" />
-        </joint>
-        <link name="${robot_name}_link_ee">
-        </link>
-    </xacro:macro>
+<robot xmlns:xacro="http://ros.org/wiki/xacro" name="apple">
+  <link name="apple_link">
+    <visual>
+      <geometry>
+        <sphere radius="0.04"/>
+      </geometry>
+      <material name="red">
+        <color rgba="1 0 0 1"/>
+      </material>
+    </visual>
+    <collision>
+      <geometry>
+        <sphere radius="0.04"/>
+      </geometry>
+    </collision>
+    <inertial>
+      <mass value="0.1"/>
+      <origin xyz="0 0 0"/>
+      <inertia ixx="0.0001" ixy="0" ixz="0" iyy="0.0001" iyz="0" izz="0.0001"/>
+    </inertial>
+  </link>
 </robot>
