Commit message: removed duplicated iiwa7 description

File: kuka_description/urdf/iiwa7_apple/iiwa7_apple.xacro (robot description, xacro)
@@ -2,29 +2,6 @@
 <!-- top level -->
 <robot name="iiwa7" xmlns:xacro="http://www.ros.org/wiki/xacro">
-    <!-- include the lbr iiwa macro -->
-    <xacro:include filename="$(find lbr_description)/urdf/iiwa7/iiwa7_description.xacro" />
-    <xacro:arg name="robot_name" default="lbr" />
-    <xacro:arg name="mode" default="mock" />
-    <xacro:arg
-        name="system_config_path"
-        default="$(find lbr_description)/ros2_control/lbr_system_config.yaml" />
-    <xacro:arg
-        name="initial_joint_positions_path"
-        default="$(find lbr_description)/ros2_control/initial_joint_positions.yaml" />
-    <!-- KDL requires a link without inertia / Gazebo requires a connection to world link or robot
-    will tipple https://github.com/lbr-stack/lbr_fri_ros2_stack/issues/230 -->
-    <link name="world" />
-    <!--joint
-        between <robot_name>_world_link and robot_name_link_0-->
-    <joint name="$(arg robot_name)_world_joint" type="fixed">
-        <parent link="world" />
-        <child link="$(arg robot_name)_link_0" />
-    </joint>
-    <!-- iiwa -->
-    <xacro:iiwa7
-        robot_name="$(arg robot_name)"
-        mode="$(arg mode)"
-        system_config_path="$(arg system_config_path)"
-        initial_joint_positions_path="$(arg initial_joint_positions_path)" />
+    <!-- include upstream top-level iiwa7 definition (adds world, base joint, and instantiates iiwa) -->
+    <xacro:include filename="$(find lbr_description)/urdf/iiwa7/iiwa7.xacro" />
     <!-- including an apple model at end of arm -->
     <xacro:include filename="$(find sinthlab_lbr_description)/urdf/models/apple.xacro"/>
